File: pcb/eagle/micromod-fc.sch (EAGLE design)
At the start: 41 parts, among them J11 microSD, J12 SM06B-GHS-TB(LF)(SN), J2 JTAG, J3 QWIIC_RIGHT_ANGLE, J4 MICROMOD-2222-C, J7 SM08B-GHS-TB(LF)(SN), U5 AP7361C-33FGE

Commit message: rev1
Parts:
- added J5: SM04B-GHS-TB(LF)(SN)-, SM04B-GHS-TB_LF__SN_-:SM04B-GHS-TB(LF)(SN)-
Connections:
- net N$24 renamed VOLTAGE
- net N$25 renamed CURRENT
- removed net A0: J4.A0
- removed net A1: J4.A1
- removed net N$13: J7.2
- removed net N$15: J7.3
- removed net N$17: J7.5
- removed net N$18: J7.6
- removed net N$19: J7.7
- removed net N$20: J7.8
- removed net N$21: J12.SHIELD
- removed net N$22: J12.6
- removed net N$23: J12.5
- removed net N$26: J12.2
- removed net N$27: J12.1
- removed net PWM0: J4.PWM0
- removed net PWM1/CAM_VDD: J4.PWM1
- new net ESC_TELEM: J4.RX2, J7.2
- new net M1: J4.A0, J7.5
- new net M2: J4.A1, J7.6
- new net M3: J4.PWM0, J7.7
- new net M4: J4.PWM1, J7.8
- new net VRAW: J12.1, J12.2
- net 3.3V: now also J5.1
- net GND: now also J12.5, J12.6, J12.SHIELD, J5.4, J5.SHIELD, J7.3
- net RX1: now also J5.3
- net TX1: now also J5.2
Changed lines of the file:
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@@
 <part name="J7" library="SM08B-GHS-TB_LF__SN_" deviceset="SM08B-GHS-TB(LF)(SN)" device=""/>
 <part name="J12" library="SM06B-GHS-TB_LF__SN_" deviceset="SM06B-GHS-TB(LF)(SN)" device=""/>
+<part name="J5" library="SM04B-GHS-TB_LF__SN_-" deviceset="SM04B-GHS-TB(LF)(SN)-" device=""/>
 </parts>
 <sheets>
@@
 <attribute name="VALUE" x="233.68" y="147.32" size="1.778" layer="96"/>
 </instance>
+<instance part="J5" gate="G$1" x="236.22" y="127" smashed="yes">
+<attribute name="NAME" x="231.13978125" y="134.62033125" size="1.27005" layer="95"/>
+<attribute name="VALUE" x="231.13411875" y="114.2853" size="1.27146875" layer="96"/>
+</instance>
 </instances>
 <busses>
@@
 <wire x1="228.6" y1="185.42" x2="213.36" y2="185.42" width="0.1524" layer="91"/>
 <label x="213.36" y="185.42" size="1.778" layer="95"/>
+</segment>
+<segment>
+<pinref part="J7" gate="G$1" pin="3"/>
+<wire x1="228.6" y1="203.2" x2="213.36" y2="203.2" width="0.1524" layer="91"/>
+<label x="213.36" y="203.2" size="1.778" layer="95"/>
+</segment>
+<segment>
+<pinref part="J12" gate="G$1" pin="5"/>
+<wire x1="228.6" y1="160.02" x2="215.9" y2="160.02" width="0.1524" layer="91"/>
+<label x="215.9" y="160.02" size="1.778" layer="95"/>
+</segment>
+<segment>
+<pinref part="J12" gate="G$1" pin="6"/>
+<wire x1="228.6" y1="157.48" x2="223.52" y2="157.48" width="0.1524" layer="91"/>
+<label x="215.9" y="157.48" size="1.778" layer="95"/>
+<pinref part="J12" gate="G$1" pin="SHIELD"/>
+<wire x1="223.52" y1="157.48" x2="215.9" y2="157.48" width="0.1524" layer="91"/>
+<wire x1="228.6" y1="152.4" x2="223.52" y2="152.4" width="0.1524" layer="91"/>
+<wire x1="223.52" y1="152.4" x2="215.9" y2="152.4" width="0.1524" layer="91"/>
+<wire x1="223.52" y1="157.48" x2="223.52" y2="152.4" width="0.1524" layer="91"/>
+<junction x="223.52" y="157.48"/>
+<junction x="223.52" y="152.4"/>
+</segment>
+<segment>
+<pinref part="J5" gate="G$1" pin="4"/>
+<wire x1="226.06" y1="124.46" x2="215.9" y2="124.46" width="0.1524" layer="91"/>
+<label x="215.9" y="124.46" size="1.778" layer="95"/>
+</segment>
+<segment>
+<pinref part="J5" gate="G$1" pin="SHIELD"/>
+<wire x1="226.06" y1="119.38" x2="215.9" y2="119.38" width="0.1524" layer="91"/>
+<label x="215.9" y="119.38" size="1.778" layer="95"/>
 </segment>
 </net>
@@
 <wire x1="152.4" y1="266.7" x2="152.4" y2="269.24" width="0.1524" layer="91"/>
 </segment>
+<segment>
+<pinref part="J5" gate="G$1" pin="1"/>
+<wire x1="226.06" y1="132.08" x2="215.9" y2="132.08" width="0.1524" layer="91"/>
+<label x="218.44" y="132.08" size="1.778" layer="95"/>
+</segment>
 </net>
 <net name="USB_D-" class="0">
@@
 <pinref part="J4" gate="J1" pin="TX1"/>
 </segment>
+<segment>
+<pinref part="J5" gate="G$1" pin="2"/>
+<wire x1="226.06" y1="129.54" x2="215.9" y2="129.54" width="0.1524" layer="91"/>
+<label x="215.9" y="129.54" size="1.778" layer="95"/>
+</segment>
 </net>
 <net name="RX1" class="0">
@@
 <label x="137.16" y="76.2" size="1.27" layer="95" xref="yes"/>
 <pinref part="J4" gate="J1" pin="RX1"/>
+</segment>
+<segment>
+<pinref part="J5" gate="G$1" pin="3"/>
+<wire x1="226.06" y1="127" x2="215.9" y2="127" width="0.1524" layer="91"/>
+<label x="215.9" y="127" size="1.778" layer="95"/>
 </segment>
 </net>
@@
 </segment>
 </net>
-<net name="A0" class="0">
-<segment>
-<wire x1="134.62" y1="96.52" x2="137.16" y2="96.52" width="0.1524" layer="91"/>
-<label x="137.16" y="96.52" size="1.27" layer="95" xref="yes"/>
-<pinref part="J4" gate="J1" pin="A0"/>
-</segment>
-</net>
-<net name="A1" class="0">
-<segment>
-<wire x1="134.62" y1="93.98" x2="137.16" y2="93.98" width="0.1524" layer="91"/>
-<label x="137.16" y="93.98" size="1.27" layer="95" xref="yes"/>
-<pinref part="J4" gate="J1" pin="A1"/>
-</segment>
-</net>
-<net name="PWM0" class="0">
-<segment>
-<wire x1="134.62" y1="91.44" x2="137.16" y2="91.44" width="0.1524" layer="91"/>
-<label x="137.16" y="91.44" size="1.27" layer="95" xref="yes"/>
-<pinref part="J4" gate="J1" pin="PWM0"/>
-</segment>
-</net>
-<net name="PWM1/CAM_VDD" class="0">
+<net name="M4" class="0">
 <segment>
 <wire x1="134.62" y1="88.9" x2="137.16" y2="88.9" width="0.1524" layer="91"/>
 <label x="137.16" y="88.9" size="1.27" layer="95" xref="yes"/>
 <pinref part="J4" gate="J1" pin="PWM1"/>
+</segment>
+<segment>
+<pinref part="J7" gate="G$1" pin="8"/>
+<wire x1="228.6" y1="190.5" x2="213.36" y2="190.5" width="0.1524" layer="91"/>
+<label x="213.36" y="190.5" size="1.778" layer="95"/>
 </segment>
 </net>
@@
 </segment>
 </net>
-<net name="N$13" class="0">
+<net name="ESC_TELEM" class="0">
 <segment>
 <pinref part="J7" gate="G$1" pin="2"/>
 <wire x1="228.6" y1="205.74" x2="213.36" y2="205.74" width="0.1524" layer="91"/>
-</segment>
-</net>
-<net name="N$15" class="0">
-<segment>
-<pinref part="J7" gate="G$1" pin="3"/>
-<wire x1="228.6" y1="203.2" x2="213.36" y2="203.2" width="0.1524" layer="91"/>
+<label x="213.36" y="205.74" size="1.778" layer="95"/>
+</segment>
+<segment>
+<pinref part="J4" gate="J1" pin="RX2"/>
+<wire x1="134.62" y1="66.04" x2="144.78" y2="66.04" width="0.1524" layer="91"/>
+<label x="144.78" y="66.04" size="1.778" layer="95"/>
 </segment>
 </net>
@@
 </segment>
 </net>
-<net name="N$17" class="0">
+<net name="M1" class="0">
 <segment>
 <pinref part="J7" gate="G$1" pin="5"/>
 <wire x1="228.6" y1="198.12" x2="213.36" y2="198.12" width="0.1524" layer="91"/>
-</segment>
-</net>
-<net name="N$18" class="0">
+<label x="213.36" y="198.12" size="1.778" layer="95"/>
+</segment>
+<segment>
+<wire x1="134.62" y1="96.52" x2="137.16" y2="96.52" width="0.1524" layer="91"/>
+<label x="137.16" y="96.52" size="1.27" layer="95" xref="yes"/>
+<pinref part="J4" gate="J1" pin="A0"/>
+</segment>
+</net>
+<net name="M2" class="0">
 <segment>
 <pinref part="J7" gate="G$1" pin="6"/>
 <wire x1="228.6" y1="195.58" x2="213.36" y2="195.58" width="0.1524" layer="91"/>
-</segment>
-</net>
-<net name="N$19" class="0">
+<label x="213.36" y="195.58" size="1.778" layer="95"/>
+</segment>
+<segment>
+<wire x1="134.62" y1="93.98" x2="137.16" y2="93.98" width="0.1524" layer="91"/>
+<label x="137.16" y="93.98" size="1.27" layer="95" xref="yes"/>
+<pinref part="J4" gate="J1" pin="A1"/>
+</segment>
+</net>
+<net name="M3" class="0">
 <segment>
 <pinref part="J7" gate="G$1" pin="7"/>
 <wire x1="228.6" y1="193.04" x2="213.36" y2="193.04" width="0.1524" layer="91"/>
-</segment>
-</net>
-<net name="N$20" class="0">
-<segment>
-<pinref part="J7" gate="G$1" pin="8"/>
-<wire x1="228.6" y1="190.5" x2="213.36" y2="190.5" width="0.1524" layer="91"/>
-</segment>
-</net>
-<net name="N$21" class="0">
-<segment>
-<pinref part="J12" gate="G$1" pin="SHIELD"/>
-<wire x1="228.6" y1="152.4" x2="215.9" y2="152.4" width="0.1524" layer="91"/>
-</segment>
-</net>
-<net name="N$22" class="0">
-<segment>
-<pinref part="J12" gate="G$1" pin="6"/>
-<wire x1="228.6" y1="157.48" x2="215.9" y2="157.48" width="0.1524" layer="91"/>
-</segment>
-</net>
-<net name="N$23" class="0">
-<segment>
-<pinref part="J12" gate="G$1" pin="5"/>
-<wire x1="228.6" y1="160.02" x2="215.9" y2="160.02" width="0.1524" layer="91"/>
-</segment>
-</net>
-<net name="N$24" class="0">
+<label x="213.36" y="193.04" size="1.778" layer="95"/>
+</segment>
+<segment>
+<wire x1="134.62" y1="91.44" x2="137.16" y2="91.44" width="0.1524" layer="91"/>
+<label x="137.16" y="91.44" size="1.27" layer="95" xref="yes"/>
+<pinref part="J4" gate="J1" pin="PWM0"/>
+</segment>
+</net>
+<net name="VRAW" class="0">
+<segment>
+<pinref part="J12" gate="G$1" pin="1"/>
+<wire x1="228.6" y1="170.18" x2="215.9" y2="170.18" width="0.1524" layer="91"/>
+<label x="215.9" y="170.18" size="1.778" layer="95"/>
+</segment>
+<segment>
+<pinref part="J12" gate="G$1" pin="2"/>
+<wire x1="228.6" y1="167.64" x2="215.9" y2="167.64" width="0.1524" layer="91"/>
+<label x="215.9" y="167.64" size="1.778" layer="95"/>
+</segment>
+</net>
+<net name="VOLTAGE" class="0">
 <segment>
 <pinref part="J12" gate="G$1" pin="4"/>
 <wire x1="228.6" y1="162.56" x2="215.9" y2="162.56" width="0.1524" layer="91"/>
-</segment>
-</net>
-<net name="N$25" class="0">
+<label x="215.9" y="162.56" size="1.778" layer="95"/>
+</segment>
+</net>
+<net name="CURRENT" class="0">
 <segment>
 <pinref part="J12" gate="G$1" pin="3"/>
 <wire x1="228.6" y1="165.1" x2="215.9" y2="165.1" width="0.1524" layer="91"/>
-</segment>
-</net>
-<net name="N$26" class="0">
-<segment>
-<pinref part="J12" gate="G$1" pin="2"/>
-<wire x1="228.6" y1="167.64" x2="215.9" y2="167.64" width="0.1524" layer="91"/>
-</segment>
-</net>
-<net name="N$27" class="0">
-<segment>
-<pinref part="J12" gate="G$1" pin="1"/>
-<wire x1="228.6" y1="170.18" x2="215.9" y2="170.18" width="0.1524" layer="91"/>
-</segment>
-</net>
+<label x="215.9" y="165.1" size="1.778" layer="95"/>
+</segment>
+</net>

Commit message: rev1.1.
Parts:
- added J10: (no value), SparkFun-Connectors:CONN_01
- added J8: (no value), SparkFun-Connectors:CONN_03
Connections:
- net 3.3V: now also J10.1
- net GND: now also J8.1
- net I2C_SCL: now also J8.2
- net I2C_SDA: now also J8.3
Changed lines of the file:
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@@
 <part name="J12" library="SM06B-GHS-TB_LF__SN_" deviceset="SM06B-GHS-TB(LF)(SN)" device=""/>
 <part name="J5" library="SM04B-GHS-TB_LF__SN_-" deviceset="SM04B-GHS-TB(LF)(SN)-" device=""/>
+<part name="J10" library="SparkFun-Connectors" library_urn="urn:adsk.eagle:library:513" deviceset="CONN_01" device="" package3d_urn="urn:adsk.eagle:package:38028/1"/>
+<part name="J8" library="SparkFun-Connectors" library_urn="urn:adsk.eagle:library:513" deviceset="CONN_03" device="" package3d_urn="urn:adsk.eagle:package:38063/1"/>
 </parts>
 <sheets>
@@
 <attribute name="VALUE" x="231.13411875" y="114.2853" size="1.27146875" layer="96"/>
 </instance>
+<instance part="J10" gate="G$1" x="226.06" y="40.64" smashed="yes" rot="R180">
+<attribute name="VALUE" x="228.6" y="45.466" size="1.778" layer="96" font="vector" rot="R180"/>
+<attribute name="NAME" x="228.6" y="37.592" size="1.778" layer="95" font="vector" rot="R180"/>
+</instance>
+<instance part="J8" gate="J$1" x="228.6" y="30.48" smashed="yes" rot="R180">
+<attribute name="VALUE" x="231.14" y="37.846" size="1.778" layer="96" font="vector" rot="R180"/>
+<attribute name="NAME" x="231.14" y="24.892" size="1.778" layer="95" font="vector" rot="R180"/>
+</instance>
 </instances>
 <busses>
@@
 <wire x1="226.06" y1="119.38" x2="215.9" y2="119.38" width="0.1524" layer="91"/>
 <label x="215.9" y="119.38" size="1.778" layer="95"/>
+</segment>
+<segment>
+<wire x1="220.98" y1="33.02" x2="205.74" y2="33.02" width="0.1524" layer="91"/>
+<pinref part="J8" gate="J$1" pin="1"/>
+<label x="213.36" y="33.02" size="1.778" layer="95"/>
 </segment>
 </net>
@@
 <label x="218.44" y="132.08" size="1.778" layer="95"/>
 </segment>
+<segment>
+<pinref part="J10" gate="G$1" pin="1"/>
+<wire x1="218.44" y1="40.64" x2="205.74" y2="40.64" width="0.1524" layer="91"/>
+<label x="210.82" y="40.64" size="1.778" layer="95"/>
+</segment>
 </net>
 <net name="USB_D-" class="0">
@@
 <pinref part="J4" gate="J1" pin="I2C_SCL"/>
 </segment>
+<segment>
+<wire x1="220.98" y1="30.48" x2="205.74" y2="30.48" width="0.1524" layer="91"/>
+<label x="205.74" y="30.48" size="1.778" layer="95"/>
+<pinref part="J8" gate="J$1" pin="2"/>
+</segment>
 </net>
 <net name="I2C_SDA" class="0">
@@
 <label x="86.36" y="58.42" size="1.27" layer="95" rot="MR0" xref="yes"/>
 <pinref part="J4" gate="J1" pin="I2C_SDA"/>
+</segment>
+<segment>
+<wire x1="220.98" y1="27.94" x2="205.74" y2="27.94" width="0.1524" layer="91"/>
+<label x="205.74" y="27.94" size="1.778" layer="95"/>
+<pinref part="J8" gate="J$1" pin="3"/>
 </segment>
 </net>
@@
 which will not be processed correctly with this version.
 </note>
+<note version="8.2" severity="warning">
+Since Version 8.2, EAGLE supports online libraries. The ids
+of those online libraries will not be understood (or retained)
+with this version.
+</note>
 <note version="8.3" severity="warning">
