File: pcb/eagle/micromod-fc.brd (EAGLE design)
At the start: 36 x 36 mm, 41 parts, among them J11 microSD, J12 SM06B-GHS-TB(LF)(SN), J2 JTAG, J3 QWIIC_RIGHT_ANGLE, J4 MICROMOD-2222-C, J7 SM08B-GHS-TB(LF)(SN), U5 AP7361C-33FGE

Commit message: rev1
Parts:
- added J5: SM04B-GHS-TB(LF)(SN)-, SM04B-GHS-TB_LF__SN_-:JST_SM04B-GHS-TB(LF)(SN)-
Connections:
- net N$24 renamed VOLTAGE
- net N$25 renamed CURRENT
- removed net A0: J4.34
- removed net A1: J4.38
- removed net N$13: J7.2
- removed net N$15: J7.3
- removed net N$17: J7.5
- removed net N$18: J7.6
- removed net N$19: J7.7
- removed net N$20: J7.8
- removed net N$21: J12.S1, J12.S2
- removed net N$22: J12.6
- removed net N$23: J12.5
- removed net N$26: J12.2
- removed net N$27: J12.1
- removed net PWM0: J4.32
- removed net PWM1/CAM_VDD: J4.47
- new net ESC_TELEM: J4.20, J7.2
- new net M1: J4.34, J7.5
- new net M2: J4.38, J7.6
- new net M3: J4.32, J7.7
- new net M4: J4.47, J7.8
- new net VRAW: J12.1, J12.2
- net 3.3V: now also J5.1
- net GND: now also J12.5, J12.6, J12.S1, J12.S2, J5.4, J5.SH1, J5.SH2, J7.3
- net RX1: now also J5.3
- net TX1: now also J5.2
Routing:
- net 3.3V: track 73.9 -> 149.7 mm, vias 5 -> 11
- net M1: track 0.00 -> 57.4 mm, vias 0 -> 4
- net M2: track 0.00 -> 54.9 mm, vias 0 -> 4
- net M3: track 0.00 -> 51.5 mm, vias 0 -> 4
- net GND: track 182.7 -> 233.9 mm, vias 4 -> 10
- net M4: track 0.00 -> 44.9 mm, vias 0 -> 2
- net ESC_TELEM: track 0.00 -> 12.4 mm, vias 0 -> 2
- net N$21: track 9.95 -> 0.00 mm
- net N$2: track 0.00 -> 9.88 mm, vias 0 -> 2
- net RTC_3V: track 20.5 -> 29.2 mm, vias 1 -> 2
- net VIN/3: track 22.7 -> 28.7 mm
- net VIN: track 59.7 -> 62.7 mm, vias 2 -> 3
- net VREG_3.3V: track 24.1 -> 26.3 mm
- net I2C_SCL: track 17.0 -> 19.0 mm
- net !BOOT!: track 13.5 -> 15.0 mm
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
Commit message: rev1.1.
Parts:
- added J10: (no value), SparkFun-Connectors:1X01
- added J8: (no value), SparkFun-Connectors:1X03
- moved J5 42.8 mm to (32.5, 12.0), flipped to the bottom, turned to 270 degrees
- moved VIN_LED 1.50 mm to (10.2, 14.2)
Connections:
- net 3.3V: now also J10.1
- net GND: now also J8.1
- net I2C_SCL: now also J8.2
- net I2C_SDA: now also J8.3
Routing:
- net GND: track 233.9 -> 278.0 mm, vias 10 -> 11
- net 3.3V: track 149.7 -> 184.0 mm, vias 11 -> 13
- net I2C_SDA: track 18.5 -> 50.7 mm, vias 2 -> 6
- net I2C_SCL: track 19.0 -> 38.1 mm, vias 2 -> 6
- net VREG_3.3V: track 26.3 -> 43.7 mm
- net RX1: track 0.00 -> 15.1 mm, vias 0 -> 1
- net TX1: track 0.00 -> 12.9 mm, vias 0 -> 1
- net USB_D-: track 27.4 -> 33.2 mm
- net VIN/3: track 28.7 -> 33.7 mm
- net SWDIO: track 28.8 -> 33.5 mm
- net M4: track 44.9 -> 47.9 mm
- net 3.3V_EN: track 16.0 -> 18.6 mm
- net M3: track 51.5 -> 53.8 mm
- net M1: track 57.4 -> 59.7 mm
- net N$14: track 42.2 -> 44.1 mm
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
Commit message: maybe new
Routing:
- net VREG_3.3V: track 43.7 -> 38.4 mm
Changed lines of the file:
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@@
 <attribute name="PACKAGE" value="None" x="32.5" y="12" size="1.778" layer="28" rot="MR270" display="off"/>
 <attribute name="PURCHASE-URL" value="https://pricing.snapeda.com/search/part/SM04B-GHS-TB(LF)(SN)-/?ref=eda" x="32.5" y="12" size="1.778" layer="28" rot="MR270" display="off"/>
-<attribute name="VALUE" x="36.50248125" y="16.502790625" size="1.270790625" layer="28" rot="MR270"/>
 </element>
 <element name="J10" library="SparkFun-Connectors" library_urn="urn:adsk.eagle:library:513" package="1X01" package3d_urn="urn:adsk.eagle:package:38028/1" value="" x="12.75" y="19.25" smashed="yes">
@@
 <wire x1="30.0054" y1="20.9744" x2="30" y2="20.969" width="0.1524" layer="1"/>
 <wire x1="30.215" y1="20.535" x2="29.75" y2="21" width="0.1524" layer="16"/>
+<wire x1="32.26" y1="28.74" x2="32.1876" y2="28.74" width="0.1524" layer="1"/>
+<wire x1="32.1876" y1="28.74" x2="32.0526" y2="28.875" width="0.1524" layer="1"/>
 </signal>
 <signal name="3.3V">
@@
 <wire x1="33.40205" y1="19.8932" x2="33.90475" y2="19.8932" width="0.1524" layer="16"/>
 <wire x1="32.03505" y1="19.8932" x2="33.40205" y2="19.8932" width="0.1524" layer="16"/>
-<wire x1="34.5186" y1="25.8296875" x2="33.6846875" y2="26.6636" width="0.1524" layer="16"/>
 <wire x1="28.8416" y1="16.69975" x2="32.03505" y2="19.8932" width="0.1524" layer="16"/>
-<wire x1="33.6846875" y1="26.6636" x2="32.535" y2="26.6636" width="0.1524" layer="16"/>
-<wire x1="32.535" y1="26.6636" x2="30.4486" y2="28.75" width="0.1524" layer="16"/>
 <wire x1="33.90475" y1="19.8932" x2="34.5186" y2="20.50705" width="0.1524" layer="16"/>
 <wire x1="34.5186" y1="20.50705" x2="34.5186" y2="25.8296875" width="0.1524" layer="16"/>
